File: sim/discharge/discharge.kicad_sch (KiCad schematic)
At the start: 9 parts, among them Q1 NMOS

Commit message: Save bms sim
Parts:
- D1: value D -> 1N4148W
- Q1: value NMOS -> AO3400
Changed lines of the file:
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@@
 			)
 		)
-		(property "Value" "NMOS"
+		(property "Value" "AO3400"
 			(at 91.44 64.7699 0)
 			(effects
@@
 			)
 		)
-		(property "Sim.Library" "ao3400.spice"
+		(property "Sim.Library" "/home/miguel/Projects/kicad-lib/spice/ao3400.spice"
 			(at 97.79 63.5 0)
 			(effects
@@
 		(on_board yes)
 		(dnp no)
-		(fields_autoplaced yes)
 		(property "Reference" "D1"
-			(at 118.11 68.5799 90)
-			(effects
-				(font
-					(size 1.27 1.27)
-				)
-				(justify left)
-			)
-		)
-		(property "Value" "D"
-			(at 118.11 71.1199 90)
+			(at 116.586 73.66 90)
+			(effects
+				(font
+					(size 1.27 1.27)
+				)
+				(justify left)
+			)
+		)
+		(property "Value" "1N4148W"
+			(at 109.728 77.978 90)
 			(effects
 				(font
@@
 			)
 		)
-		(property "Sim.Library" "1n4148w.spice"
+		(property "Sim.Library" "/home/miguel/Projects/kicad-lib/spice/1n4148w.spice"
 			(at 115.57 69.85 0)
 			(effects
@@
 			(at 115.57 69.85 0)
 			(effects
+				(font
+					(size 1.27 1.27)
+				)
+				(hide yes)
+			)
+		)
+		(property "Sim.Params" "temp=25"
+			(at 115.57 69.85 0)
+			(effects
