File: sim/regulator/regulator.kicad_sch (KiCad schematic)
At the start: 0 parts

Commit message: Save
Parts:
- added C1: 100n ic=0, symbol Device:C
- added C11, C12: 4.7u ic=0, symbol Device:C
- added C13: 443p ic=0, symbol Device:C
- added C14: 5n ic=0, symbol Device:C
- added C15: 126.9n ic=1.2, symbol Device:C
- added C2: 100n, symbol Device:C
- added C3: 10u, Resistor_SMD:R_0603_1608Metric, symbol Device:C
- added C7: 58p ic=0, symbol Device:C
- added D1, D2, D3, D4: 1N4148W, symbol Simulation_SPICE:D
- added L1: 330u ic=0, symbol Device:L
- added Q1, Q7: PNP, symbol Simulation_SPICE:PNP
- added Q10, Q11, Q2, Q4, Q6, Q8, Q9: NPN, symbol Simulation_SPICE:NPN
- added Q3, Q5: NMOS, symbol Simulation_SPICE:NMOS
- added R1, R17, R19: 10k, symbol Device:R
- added R10: 20k, symbol Device:R
- added R11: 80k, symbol Device:R
- added R12, R14: 47k, symbol Device:R
- added R13: 63k, symbol Device:R
- added R15, R16, R18, R20, R9: 2k, symbol Device:R
- added R2: 8.2k, symbol Device:R
- added R21: 1k, symbol Device:R
- added R3: 70, symbol Device:R
- added R34: 40, symbol Device:R
- added R35: 42857, symbol Device:R
- added R36: 100k, symbol Device:R
- added R37: 4k, symbol Device:R
- added R38: 350, symbol Device:R
- added R4: 30k, symbol Device:R
- added R5, R6: 100, symbol Device:R
- added R7: 2, symbol Device:R
- added R8: 200m, symbol Device:R
- added S1, S2: SWITCH, symbol Simulation_SPICE:SWITCH
- added U1, U10, U2, U3, U5, U6, U7, U8: ${SIM.PARAMS}, symbol Simulation_SPICE:OPAMP
- added U4: HT7533-1-SOT89, Package_TO_SOT_SMD:SOT-89-3, symbol Regulator_Linear:HT75xx-1-SOT89
- added U9: LMV7219M5, Package_TO_SOT_SMD:SOT-23-5, symbol Comparator:LMV7219M5
- added V1, V3, V4, V8: VPULSE, symbol Simulation_SPICE:VPULSE
- added V2: 0.25, symbol Simulation_SPICE:VDC
- added V5: 3.3, symbol Simulation_SPICE:VDC
- added V6: 5, symbol Simulation_SPICE:VDC
- added V7: 65, symbol Simulation_SPICE:VDC
Connections:
- new net: D2.2 (A), D3.2 (A), S1.1 (N+)
- new net: Q10.1 (C), Q9.2 (B), R19.1
- new net: C7.2, R13.1, U7.2 (-)
- new net: U10.2 (-), V2.1
- new net: Q1.3 (E), Q2.3 (E), Q3.2 (G)
- new net: R10.1, R11.1, U8.1 (+)
- new net: C14.1, R35.1, R36.2, R37.2, R38.1, U1.2 (-)
- new net: Q6.2 (B), Q7.2 (B), R6.2
- new net: Q10.2 (B), R20.2
- new net: Q11.1 (C), Q8.2 (B), R17.2
- new net: R12.1, R9.2, U5.1 (+)
- new net: R3.2, S2.1 (N+)
- new net: C15.1, R38.2
- new net: Q8.1 (C), R18.2, R19.2
- new net: R7.2, V6.1
- new net: R7.1, S1.2 (N-)
- new net: Q11.2 (B), R21.1
- new net: R21.2, V8.1
- new net: R14.2, R15.1, U5.2 (-)
- new net: S1.3 (C+), V4.1
- new net: C13.2, R37.1
- new net: Q1.2 (B), Q2.2 (B), Q4.1 (C), R4.2
- new net: Q4.2 (B), R5.2
- new net +3V3: C3.1, R1.1, U1.3 (V+), U2.3 (V+), U4.3 (VOUT), U7.3 (V+), U8.3 (V+), V5.1
- new net +5V: C2.1, D1.2 (A), D3.1 (K), D4.1 (K), Q6.1 (C), R15.2, R16.1, R18.1, R3.1, U10.3 (V+), U4.2 (VIN), U5.3 (V+)
- new net 0: C11.2, C12.2, C13.1, C2.2, C3.2, Q1.1 (C), Q10.3 (E), Q11.3 (E), Q4.3 (E), Q5.3 (S), Q7.1 (C), Q8.3 (E), Q9.3 (E), R12.2, R2.2, R34.2, R35.2, R36.1, S1.4 (C-), S2.2 (N-), S2.4 (C-), U1.4 (V-), U10.4 (V-), U2.4 (V-), U4.1 (GND), U5.4 (V-), U7.4 (V-), U8.4 (V-), V1.2, V2.2, V3.2, V4.2, V5.2, V6.2, V7.2, V8.2
- new net BOOT: C1.1, D1.1 (K), Q2.1 (C), R4.1
- new net G: Q5.2 (G), Q6.3 (E), Q7.3 (E)
- new net IGAIN: R14.1, U10.1 (+), U5.5
- new net IND: L1.2, R8.1, R9.1
- new net L: S2.3 (C+), V3.1
- new net P5: C11.1, C12.1, D4.2 (A), R34.1, R8.2
- new net PWM: D2.1 (K), Q9.1 (C), R16.2, R17.1, R5.1, R6.1
- new net Q: R20.1, U10.5
- new net REF: C14.2, C15.2, U1.5, U2.2 (-)
- new net SQ: R11.2, R13.2, U8.5
- new net SW: C1.2, L1.1, Q3.3 (S), Q5.1 (D)
- new net TR: U2.1 (+), V1.1
- new net TR2: C7.1, R10.2, U7.5
- new net VBAT: Q3.1 (D), V7.1
- new net VD2: R1.2, R2.1, U1.1 (+), U7.1 (+), U8.2 (-)
Other:
- note added: "1uF is enough for 50mV ripple, but >=10uF for stability"
- note added: "2x 1206 4.7uF X7R"
- note added: "L = 330uH"
- note added: "Ripple < 40%"
- note added: "ZXMP10A13FPA"
- note added: "f_sw = 200khz"
- note added: "state space averaging"
- note added: "type II controller for voltage"
