File: pcb/battery-pack.kicad_pcb (KiCad board)
At the start: 4 copper layers, 0 parts

Commit message: Save bms descrete prototype
Parts:
- added C18: 100n, Capacitor_SMD:C_0805_2012Metric, F.Cu at (179.0, 62.0)
- added C19: 100n, Capacitor_SMD:C_0805_2012Metric, F.Cu at (189.7, 59.6)
- added C20: 100n, Capacitor_SMD:C_0805_2012Metric, F.Cu at (100.5, 49.4)
- added C21: 100n, Capacitor_SMD:C_0805_2012Metric, F.Cu at (188.0, 62.0)
- added C24: 100n, Capacitor_SMD:C_0805_2012Metric, F.Cu at (100.5, 55.4)
- added C27: 100n, Capacitor_SMD:C_0805_2012Metric, F.Cu at (100.5, 58.4)
- added C30: 100n, Resistor_SMD:R_0603_1608Metric, F.Cu at (89.5, 63.8)
- added D1: 1N5819WS, Diode_SMD:D_SOD-323, F.Cu at (181.0, 59.0)
- added D10: 1N5819WS, Diode_SMD:D_SOD-323, F.Cu at (82.6, 49.2)
- added D11: 1N5819WS, Diode_SMD:D_SOD-323, F.Cu at (82.6, 52.2)
- added D12: 1N5819WS, Diode_SMD:D_SOD-323, F.Cu at (82.6, 55.1)
- added D13: 1N5819WS, Diode_SMD:D_SOD-323, F.Cu at (82.6, 58.1)
- added D14: 1N5819WS, Diode_SMD:D_SOD-323, F.Cu at (82.6, 61.0)
- added D15: 1N5819WS, Diode_SMD:D_SOD-323, F.Cu at (86.9, 43.3)
- added D16: 1N5819WS, Diode_SMD:D_SOD-323, F.Cu at (86.9, 46.3)
- added D17: 1N5819WS, Diode_SMD:D_SOD-323, F.Cu at (86.9, 49.2)
- added D18: 1N5819WS, Diode_SMD:D_SOD-323, F.Cu at (86.9, 52.2)
- added D19: 1N5819WS, Diode_SMD:D_SOD-323, F.Cu at (86.9, 55.1)
- added D2: 1N5819WS, Diode_SMD:D_SOD-323, F.Cu at (188.5, 57.5)
- added D20: 1N5819WS, Diode_SMD:D_SOD-323, F.Cu at (86.9, 58.1)
- added D21: 1N5819WS, Diode_SMD:D_SOD-323, F.Cu at (86.9, 61.0)
- added D22: 1N5819WS, Diode_SMD:D_SOD-323, F.Cu at (91.2, 43.3)
- added D23: 1N5819WS, Diode_SMD:D_SOD-323, F.Cu at (91.2, 46.3)
- added D24: 1N5819WS, Diode_SMD:D_SOD-323, F.Cu at (91.2, 49.2)
- added D3: 1N5819WS, Diode_SMD:D_SOD-323, F.Cu at (78.3, 49.2)
- added D4: 1N5819WS, Diode_SMD:D_SOD-323, F.Cu at (176.1, 58.9)
- added D5: 1N5819WS, Diode_SMD:D_SOD-323, F.Cu at (186.5, 64.0)
- added D6: 1N5819WS, Diode_SMD:D_SOD-323, F.Cu at (183.0, 59.0)
- added D7: 1N5819WS, Diode_SMD:D_SOD-323, F.Cu at (181.0, 62.5)
- added D8: 1N5819WS, Diode_SMD:D_SOD-323, F.Cu at (82.6, 43.3)
- added D9: 1N5819WS, Diode_SMD:D_SOD-323, F.Cu at (82.6, 46.3)
- added Q1: AO3400A, Package_TO_SOT_SMD:SOT-23, F.Cu at (176.1, 61.9)
- added Q10: AO3400A, Package_TO_SOT_SMD:SOT-23, F.Cu at (95.8, 67.4)
- added Q2: AO3400A, Package_TO_SOT_SMD:SOT-23, F.Cu at (95.8, 48.9)
- added Q3: MMBT5551, Package_TO_SOT_SMD:SOT-23, F.Cu at (185.9, 59.0)
- added Q4: MMBT5401, Package_TO_SOT_SMD:SOT-23, F.Cu at (183.9, 62.5)
- added Q7: AO3400A, Package_TO_SOT_SMD:SOT-23, F.Cu at (95.8, 62.8)
- added R18: 22, Resistor_SMD:R_1206_3216Metric, F.Cu at (173.0, 60.5)
- added R19: 4k7, Resistor_SMD:R_0402_1005Metric, F.Cu at (193.0, 59.5)
- added R20: 4k7, Resistor_SMD:R_0402_1005Metric, F.Cu at (179.0, 59.0)
- added R21: 4k7, Resistor_SMD:R_0402_1005Metric, F.Cu at (191.0, 62.0)
- added R22: 4k7, Resistor_SMD:R_0402_1005Metric, F.Cu at (104.1, 48.8)
- added R23: 22, Resistor_SMD:R_1206_3216Metric, F.Cu at (101.0, 64.9)
- added R26: 4k7, Resistor_SMD:R_0402_1005Metric, F.Cu at (104.1, 50.8)
- added R27: 22, Resistor_SMD:R_1206_3216Metric, F.Cu at (101.0, 68.2)
- added R30: 4k7, Resistor_SMD:R_0402_1005Metric, F.Cu at (104.1, 52.8)
- added R31: 22, Resistor_SMD:R_1206_3216Metric, F.Cu at (101.0, 71.5)
- added U1: BQ76952, Package_QFP:TQFP-48_7x7mm_P0.5mm, F.Cu at (81.8, 68.2)

Commit message: Save
Parts:
- removed D22, D23, D24: 1N5819WS, Diode_SMD:D_SOD-323
- removed Q10: AO3400A, Package_TO_SOT_SMD:SOT-23
- removed R18: 22, Resistor_SMD:R_1206_3216Metric
- removed R19: 4k7, Resistor_SMD:R_0402_1005Metric
- added C1: 100n, Capacitor_SMD:C_0402_1005Metric, F.Cu at (224.4, 90.9)
- added C10: 100n, Capacitor_SMD:C_0402_1005Metric, F.Cu at (229.0, 114.3)
- added C11: 100n, Capacitor_SMD:C_0402_1005Metric, F.Cu at (257.9, 73.7)
- added C12: 100n, Capacitor_SMD:C_0402_1005Metric, F.Cu at (244.6, 44.8)
- added C13: 100n, Capacitor_SMD:C_0402_1005Metric, F.Cu at (244.6, 102.7)
- added C14: 100n, Capacitor_SMD:C_0402_1005Metric, F.Cu at (257.9, 88.2)
- added C15: 100n, Capacitor_SMD:C_0402_1005Metric, F.Cu at (202.4, 114.3)
- added C16: 100n, Capacitor_SMD:C_0402_1005Metric, F.Cu at (257.9, 102.7)
- added C17: 100n, Capacitor_SMD:C_0402_1005Metric, F.Cu at (175.8, 114.3)
- added C2: 100p, Capacitor_SMD:C_0402_1005Metric, F.Cu at (224.4, 92.9)
- added C22: 100n, Capacitor_SMD:C_0402_1005Metric, F.Cu at (215.7, 114.3)
- added C23: 1u, Capacitor_SMD:C_0805_2012Metric, F.Cu at (200.8, 72.5)
- added C25: 100n, Capacitor_SMD:C_0402_1005Metric, F.Cu at (224.4, 94.8)
- added C26: 10u, Capacitor_SMD:C_1206_3216Metric, F.Cu at (201.4, 46.2)
- added C28: 10u, Capacitor_SMD:C_1206_3216Metric, F.Cu at (201.4, 49.6)
- added C29: 1u, Capacitor_SMD:C_0805_2012Metric, F.Cu at (200.8, 75.5)
- added C3: 1u, Capacitor_SMD:C_0805_2012Metric, F.Cu at (200.8, 69.5)
- added C31: 100p, Capacitor_SMD:C_0402_1005Metric, F.Cu at (224.4, 98.8)
- added C32: 1n, Capacitor_SMD:C_0402_1005Metric, F.Cu at (110.1, 75.1)
- added C33: 10u, Capacitor_SMD:C_1206_3216Metric, F.Cu at (201.4, 52.9)
- added C34: 10u, Capacitor_SMD:C_1206_3216Metric, F.Cu at (201.4, 56.3)
- added C35: 10u, Capacitor_SMD:C_1206_3216Metric, F.Cu at (201.4, 59.6)
- added C36: 10u, Capacitor_SMD:C_1206_3216Metric, F.Cu at (201.4, 63.0)
- added C37: 10u, Capacitor_SMD:C_1206_3216Metric, F.Cu at (201.4, 66.3)
- added C38: 10u, Capacitor_SMD:C_1206_3216Metric, F.Cu at (207.0, 36.2)
- added C39: 2u2, Capacitor_SMD:C_1206_3216Metric, F.Cu at (207.0, 39.5)
- added C40: 2u2, Capacitor_SMD:C_1206_3216Metric, F.Cu at (207.0, 42.9)
- added C41: 10u, Capacitor_SMD:C_1206_3216Metric, F.Cu at (207.0, 46.2)
- added C42: 10u, Capacitor_SMD:C_1206_3216Metric, F.Cu at (207.0, 49.6)
- added C43: 10u, Capacitor_SMD:C_1206_3216Metric, F.Cu at (207.0, 52.9)
- added C44: 10u, Capacitor_SMD:C_1206_3216Metric, F.Cu at (207.0, 56.3)
- added C45: 2u2, Capacitor_SMD:C_1206_3216Metric, F.Cu at (207.0, 59.6)
- added C46: 2u2, Capacitor_SMD:C_1206_3216Metric, F.Cu at (207.0, 63.0)
- added C47: 10u, Capacitor_SMD:C_1206_3216Metric, F.Cu at (207.0, 66.3)
- added C48: 10u, Capacitor_SMD:C_1206_3216Metric, F.Cu at (212.7, 36.2)
- added C49: 10u, Capacitor_SMD:C_1206_3216Metric, F.Cu at (212.7, 39.5)
- added C5: 2u2, Capacitor_SMD:C_1206_3216Metric, F.Cu at (201.4, 36.2)
- added C50: 10u, Capacitor_SMD:C_1206_3216Metric, F.Cu at (212.7, 42.9)
- added C51: 2u2, Capacitor_SMD:C_1206_3216Metric, F.Cu at (212.7, 46.2)
- added C52: 100n, Capacitor_SMD:C_0402_1005Metric, F.Cu at (227.3, 90.9)
- added C53: 2u2, Capacitor_SMD:C_1206_3216Metric, F.Cu at (212.7, 49.6)
- added C54: 10u, Capacitor_SMD:C_1206_3216Metric, F.Cu at (212.7, 52.9)
- added C55: 10u, Capacitor_SMD:C_1206_3216Metric, F.Cu at (212.7, 56.3)
- added C56: 10u, Capacitor_SMD:C_1206_3216Metric, F.Cu at (212.7, 59.6)
- added C57: 10u, Capacitor_SMD:C_1206_3216Metric, F.Cu at (212.7, 63.0)
- added C58: 2u2, Capacitor_SMD:C_1206_3216Metric, F.Cu at (212.7, 66.3)
- added C59: 2u2, Capacitor_SMD:C_1206_3216Metric, F.Cu at (218.3, 36.2)
- added C6: 100n, Capacitor_SMD:C_0402_1005Metric, F.Cu at (189.1, 114.3)
- added C60: 10u, Capacitor_SMD:C_1206_3216Metric, F.Cu at (218.3, 39.5)
- added C61: 10u, Capacitor_SMD:C_1206_3216Metric, F.Cu at (218.3, 42.9)
- added C62: 10u, Capacitor_SMD:C_1206_3216Metric, F.Cu at (218.3, 46.2)
- added C63: 2u2, Capacitor_SMD:C_1206_3216Metric, F.Cu at (218.3, 49.6)
- added C64: 2u2, Capacitor_SMD:C_1206_3216Metric, F.Cu at (218.3, 52.9)
- added C65: 2u2, Capacitor_SMD:C_1206_3216Metric, F.Cu at (218.3, 56.3)
- added C66: 2u2, Capacitor_SMD:C_1206_3216Metric, F.Cu at (218.3, 59.6)
- added C67: 2u2, Capacitor_SMD:C_1206_3216Metric, F.Cu at (218.3, 63.0)
- added C68: 2u2, Capacitor_SMD:C_1206_3216Metric, F.Cu at (218.3, 66.3)
- added C69: 2u2, Capacitor_SMD:C_1206_3216Metric, F.Cu at (224.0, 36.2)
- added C7: 100n, Capacitor_SMD:C_0402_1005Metric, F.Cu at (244.6, 73.7)
- added C70: 2u2, Capacitor_SMD:C_1206_3216Metric, F.Cu at (224.0, 39.5)
- added C71: 2u2, Capacitor_SMD:C_1206_3216Metric, F.Cu at (224.0, 42.9)
- added C72: 2u2, Capacitor_SMD:C_1206_3216Metric, F.Cu at (224.0, 46.2)
- added C73: 2u2, Capacitor_SMD:C_1206_3216Metric, F.Cu at (224.0, 49.6)
- added C74: 2u2, Capacitor_SMD:C_1206_3216Metric, F.Cu at (224.0, 52.9)
- added C75: 2u2, Capacitor_SMD:C_1206_3216Metric, F.Cu at (224.0, 56.3)
- added C76: 2u2, Capacitor_SMD:C_1206_3216Metric, F.Cu at (224.0, 59.6)
- added C77: 2u2, Capacitor_SMD:C_1206_3216Metric, F.Cu at (224.0, 63.0)
- added C78: 2u2, Capacitor_SMD:C_1206_3216Metric, F.Cu at (224.0, 66.3)
- added C79: 2u2, Capacitor_SMD:C_1206_3216Metric, F.Cu at (229.6, 36.2)
- added C8: 100n, Capacitor_SMD:C_0402_1005Metric, F.Cu at (257.9, 59.3)
- added C80: 2u2, Capacitor_SMD:C_1206_3216Metric, F.Cu at (229.6, 39.5)
- added C81: 2u2, Capacitor_SMD:C_1206_3216Metric, F.Cu at (229.6, 42.9)
- added C82: 2u2, Capacitor_SMD:C_1206_3216Metric, F.Cu at (229.6, 46.2)
- added C84: 2u2, Capacitor_SMD:C_1206_3216Metric, F.Cu at (229.6, 49.6)
- added C85: 2u2, Capacitor_SMD:C_1206_3216Metric, F.Cu at (229.6, 52.9)
- added C86: 10n, Capacitor_SMD:C_0402_1005Metric, F.Cu at (108.9, 76.1)
- added C87: 2n2, Capacitor_SMD:C_0402_1005Metric, F.Cu at (227.3, 94.8)
- added C9: 100n, Capacitor_SMD:C_0402_1005Metric, F.Cu at (257.9, 44.8)
- added C91: 100n, Capacitor_SMD:C_0402_1005Metric, F.Cu at (227.3, 96.8)
- added C92: 100n, Capacitor_SMD:C_0402_1005Metric, F.Cu at (227.3, 98.8)
- added C93: 10u, Capacitor_SMD:C_1206_3216Metric, F.Cu at (229.6, 56.3)
- added C94: 1u, Capacitor_SMD:C_0805_2012Metric, F.Cu at (200.8, 81.6)
- added C95: 10u, Capacitor_SMD:C_1206_3216Metric, F.Cu at (229.6, 59.6)
- added J10: Conn_01x02, User_Footprints:1x02_2.00mm_Solder, F.Cu at (234.0, 36.1)
- added L1: 4u7, Inductor_SMD:L_TechFuse_SL0420, F.Cu at (189.9, 95.7)
- added Q16: HL2300, Package_TO_SOT_SMD:SOT-23, F.Cu at (184.6, 114.2)
- added Q21: SP010N01BGHTO, Package_TO_SOT_SMD:Infineon_PG-HSOF-8-1, F.Cu at (191.1, 63.7)
- added Q24: AGM150P10D, Package_TO_SOT_SMD:TO-252-2, F.Cu at (229.9, 85.9)
- added Q25: HL2300, Package_TO_SOT_SMD:SOT-23, F.Cu at (240.1, 73.7)
- added Q26: HL2300, Package_TO_SOT_SMD:SOT-23, F.Cu at (253.4, 59.2)
- added Q27: HL2300, Package_TO_SOT_SMD:SOT-23, F.Cu at (253.4, 44.8)
- added Q28: HL2300, Package_TO_SOT_SMD:SOT-23, F.Cu at (224.5, 114.2)
- added Q29: HL2300, Package_TO_SOT_SMD:SOT-23, F.Cu at (253.4, 73.7)
- added Q30: HL2300, Package_TO_SOT_SMD:SOT-23, F.Cu at (240.1, 44.8)
- added Q31: HL2300, Package_TO_SOT_SMD:SOT-23, F.Cu at (240.1, 102.6)
- added Q32: HL2300, Package_TO_SOT_SMD:SOT-23, F.Cu at (253.4, 88.1)
- added Q33: HL2300, Package_TO_SOT_SMD:SOT-23, F.Cu at (197.9, 114.2)
- added Q34: HL2300, Package_TO_SOT_SMD:SOT-23, F.Cu at (253.4, 102.6)
- added Q35: HL2300, Package_TO_SOT_SMD:SOT-23, F.Cu at (171.3, 114.2)
- added Q36: HL2300, Package_TO_SOT_SMD:SOT-23, F.Cu at (240.1, 59.2)
- added Q37: HL2300, Package_TO_SOT_SMD:SOT-23, F.Cu at (240.1, 88.1)
- added Q38: HL2300, Package_TO_SOT_SMD:SOT-23, F.Cu at (240.1, 117.0)
- added Q39: HL2300, Package_TO_SOT_SMD:SOT-23, F.Cu at (211.2, 114.2)
- added Q5: SP010N01BGHTO, Package_TO_SOT_SMD:Infineon_PG-HSOF-8-1, F.Cu at (176.3, 87.1)
- added Q6: SP010N01BGHTO, Package_TO_SOT_SMD:Infineon_PG-HSOF-8-1, F.Cu at (191.1, 40.4)
- added Q8: SP010N01BGHTO, Package_TO_SOT_SMD:Infineon_PG-HSOF-8-1, F.Cu at (191.1, 52.0)
- added R1: 100, Resistor_SMD:R_0402_1005Metric, F.Cu at (204.4, 69.0)
- added R101: 1m, User_Footprints:R_Shunt_3921, F.Cu at (220.9, 78.3)
- added R102: 1, Resistor_SMD:R_0603_1608Metric, F.Cu at (230.7, 96.2)
- added R103: 1, Resistor_SMD:R_0603_1608Metric, F.Cu at (230.7, 98.7)
- added R104: 12k, Resistor_SMD:R_0402_1005Metric, F.Cu at (213.2, 71.0)
- added R105: 33k, Resistor_SMD:R_0402_1005Metric, F.Cu at (213.2, 73.0)
- added R106: 2k2, Resistor_SMD:R_0402_1005Metric, F.Cu at (213.2, 75.0)
- added R11: 100, Resistor_SMD:R_0402_1005Metric, F.Cu at (204.4, 71.0)
- added R12: 100, Resistor_SMD:R_0402_1005Metric, F.Cu at (204.4, 73.0)
- added R13: 8, Resistor_SMD:R_1225_3264Metric, F.Cu at (253.7, 53.0)
- added R14: 2k, Resistor_SMD:R_0402_1005Metric, F.Cu at (244.6, 68.4)
- added R15: 100, Resistor_SMD:R_0402_1005Metric, F.Cu at (257.9, 50.0)
- added R16: 100, Resistor_SMD:R_0402_1005Metric, F.Cu at (257.9, 52.0)
- added R17: 8, Resistor_SMD:R_1225_3264Metric, F.Cu at (253.7, 38.5)
- added R2: 100, Resistor_SMD:R_0402_1005Metric, F.Cu at (189.1, 105.0)
- added R24: 2k, Resistor_SMD:R_0402_1005Metric, F.Cu at (257.9, 54.0)
- added R25: 100, Resistor_SMD:R_0402_1005Metric, F.Cu at (189.1, 108.9)
- added R28: 100, Resistor_SMD:R_0402_1005Metric, F.Cu at (229.0, 105.0)
- added R29: 8, Resistor_SMD:R_1225_3264Metric, F.Cu at (224.8, 108.0)
- added R3: 8, Resistor_SMD:R_1225_3264Metric, F.Cu at (240.4, 67.4)
- added R32: 100, Resistor_SMD:R_0402_1005Metric, F.Cu at (257.9, 64.4)
- added R33: 8, Resistor_SMD:R_1225_3264Metric, F.Cu at (253.7, 67.4)
- added R34: 12k, Resistor_SMD:R_0402_1005Metric, F.Cu at (107.5, 74.8)
- added R35: 2k, Resistor_SMD:R_0402_1005Metric, F.Cu at (257.9, 66.4)
- added R36: 100, Resistor_SMD:R_0402_1005Metric, F.Cu at (257.9, 68.4)
- added R37: 22k, Resistor_SMD:R_0402_1005Metric, F.Cu at (204.4, 81.0)
- added R38: 2k, Resistor_SMD:R_0402_1005Metric, F.Cu at (207.3, 69.0)
- added R39: 100, Resistor_SMD:R_0402_1005Metric, F.Cu at (244.6, 35.5)
- added R4: 2k, Resistor_SMD:R_0402_1005Metric, F.Cu at (189.1, 106.9)
- added R40: 8, Resistor_SMD:R_1225_3264Metric, F.Cu at (240.4, 38.5)
- added R41: 2k, Resistor_SMD:R_0402_1005Metric, F.Cu at (244.6, 37.5)
- added R42: 100, Resistor_SMD:R_0402_1005Metric, F.Cu at (244.6, 39.5)
- added R43: 100, Resistor_SMD:R_0402_1005Metric, F.Cu at (244.6, 93.3)
- added R44: 8, Resistor_SMD:R_1225_3264Metric, F.Cu at (240.4, 96.4)
- added R45: 2k, Resistor_SMD:R_0402_1005Metric, F.Cu at (244.6, 95.3)
- added R46: 100, Resistor_SMD:R_0402_1005Metric, F.Cu at (244.6, 97.3)
- added R47: 100, Resistor_SMD:R_0402_1005Metric, F.Cu at (257.9, 78.9)
- added R48: 8, Resistor_SMD:R_1225_3264Metric, F.Cu at (253.7, 81.9)
- added R49: 2k, Resistor_SMD:R_0402_1005Metric, F.Cu at (257.9, 80.9)
- added R5: 100, Resistor_SMD:R_0402_1005Metric, F.Cu at (244.6, 64.4)
- added R50: 100, Resistor_SMD:R_0402_1005Metric, F.Cu at (257.9, 82.9)
- added R51: 100, Resistor_SMD:R_0402_1005Metric, F.Cu at (202.4, 105.0)
- added R52: 8, Resistor_SMD:R_1225_3264Metric, F.Cu at (198.2, 108.0)
- added R53: 2k, Resistor_SMD:R_0402_1005Metric, F.Cu at (202.4, 106.9)
- added R54: 100, Resistor_SMD:R_0402_1005Metric, F.Cu at (202.4, 108.9)
- added R55: 100, Resistor_SMD:R_0402_1005Metric, F.Cu at (257.9, 93.3)
- added R56: 8, Resistor_SMD:R_1225_3264Metric, F.Cu at (253.7, 96.4)
- added R57: 2k, Resistor_SMD:R_0402_1005Metric, F.Cu at (257.9, 95.3)
- added R58: 100, Resistor_SMD:R_0402_1005Metric, F.Cu at (257.9, 97.3)
- added R59: 100, Resistor_SMD:R_0402_1005Metric, F.Cu at (175.8, 105.0)
- added R6: 100, Resistor_SMD:R_0402_1005Metric, F.Cu at (244.6, 66.4)
- added R60: 8, Resistor_SMD:R_1225_3264Metric, F.Cu at (171.6, 108.0)
- added R61: 2k, Resistor_SMD:R_0402_1005Metric, F.Cu at (175.8, 106.9)
- added R62: 100, Resistor_SMD:R_0402_1005Metric, F.Cu at (175.8, 108.9)
- added R63: 100, Resistor_SMD:R_0402_1005Metric, F.Cu at (244.6, 50.0)
- added R64: 8, Resistor_SMD:R_1225_3264Metric, F.Cu at (240.4, 53.0)
- added R65: 2k, Resistor_SMD:R_0402_1005Metric, F.Cu at (244.6, 52.0)
- added R66: 100, Resistor_SMD:R_0402_1005Metric, F.Cu at (244.6, 54.0)
- added R67: 100, Resistor_SMD:R_0402_1005Metric, F.Cu at (244.6, 78.9)
- added R68: 8, Resistor_SMD:R_1225_3264Metric, F.Cu at (240.4, 81.9)
- added R69: 2k, Resistor_SMD:R_0402_1005Metric, F.Cu at (244.6, 80.9)
- added R70: 100, Resistor_SMD:R_0402_1005Metric, F.Cu at (244.6, 82.9)
- added R71: 100, Resistor_SMD:R_0402_1005Metric, F.Cu at (244.6, 107.8)
- added R72: 8, Resistor_SMD:R_1225_3264Metric, F.Cu at (240.4, 110.8)
- added R73: 2k, Resistor_SMD:R_0402_1005Metric, F.Cu at (244.6, 109.8)
- added R74: 100, Resistor_SMD:R_0402_1005Metric, F.Cu at (244.6, 111.8)
- added R75: 100, Resistor_SMD:R_0402_1005Metric, F.Cu at (215.7, 105.0)
- added R76: 8, Resistor_SMD:R_1225_3264Metric, F.Cu at (211.5, 108.0)
- added R77: 2k, Resistor_SMD:R_0402_1005Metric, F.Cu at (215.7, 106.9)
- added R78: 100, Resistor_SMD:R_0402_1005Metric, F.Cu at (215.7, 108.9)
- added R81: 2k, Resistor_SMD:R_0402_1005Metric, F.Cu at (207.3, 71.0)
- added R82: 2k, Resistor_SMD:R_0402_1005Metric, F.Cu at (207.3, 73.0)
- added R83: 2k, Resistor_SMD:R_0402_1005Metric, F.Cu at (207.3, 75.0)
- added R84: 2k, Resistor_SMD:R_0402_1005Metric, F.Cu at (207.3, 77.0)
- added R85: 100, Resistor_SMD:R_0402_1005Metric, F.Cu at (207.3, 79.0)
- added R86: 100, Resistor_SMD:R_0402_1005Metric, F.Cu at (207.3, 81.0)
- added R87: 100, Resistor_SMD:R_0402_1005Metric, F.Cu at (210.3, 69.0)
- added R88: 100, Resistor_SMD:R_0402_1005Metric, F.Cu at (210.3, 71.0)
- added R89: 100, Resistor_SMD:R_0402_1005Metric, F.Cu at (210.3, 73.0)
- added R90: 2k, Resistor_SMD:R_0402_1005Metric, F.Cu at (210.3, 75.0)
- added R91: 33k, Resistor_SMD:R_0402_1005Metric, F.Cu at (210.3, 77.0)
- added R92: 2k, Resistor_SMD:R_0402_1005Metric, F.Cu at (210.3, 79.0)
- added R93: 33k, Resistor_SMD:R_0402_1005Metric, F.Cu at (210.3, 81.0)
- added R94: 3m, Resistor_SMD:R_2512_6332Metric, F.Cu at (182.3, 95.3)
- added R95: 1, Resistor_SMD:R_0603_1608Metric, F.Cu at (230.7, 91.2)
- added R96: 1, Resistor_SMD:R_0603_1608Metric, F.Cu at (230.7, 93.7)
- added R97: 33k, Resistor_SMD:R_0402_1005Metric, F.Cu at (213.2, 69.0)
- added R98: 1m, User_Footprints:R_Shunt_3921, F.Cu at (220.9, 71.4)
- added U14: JW5017S, Package_TO_SOT_SMD:SOT-23-6, F.Cu at (195.7, 99.7)
- added U2: LM5116, Package_SO:HTSSOP-20-1EP_4.4x6.5mm_P0.65mm_EP3.4x6.5mm_Mask2.4x3.7mm, F.Cu at (116.0, 75.0)
- added U4: STM32C011F6Px, Package_SO:TSSOP-20_4.4x6.5mm_P0.65mm, F.Cu at (173.6, 96.9)
- added U5: AGM042N10A, Package_DFN_QFN:PQFN-8-EP_6x5mm_P1.27mm_Generic, F.Cu at (231.3, 71.4)
- added U6: SP485E, Package_SO:JEITA_SOIC-8_3.9x4.9mm_P1.27mm, F.Cu at (218.8, 85.1)
- added U7: AGM042N10A, Package_DFN_QFN:PQFN-8-EP_6x5mm_P1.27mm_Generic, F.Cu at (231.3, 78.3)
- added U8: IRS2181STR, Package_SO:JEITA_SOIC-8_3.9x4.9mm_P1.27mm, F.Cu at (218.8, 91.6)
- added U9: XC6206PxxxMR, Package_TO_SOT_SMD:SOT-23-3, F.Cu at (195.7, 95.1)
- C18: value 100n -> 10u; footprint Capacitor_SMD:C_0805_2012Metric -> Capacitor_SMD:C_1206_3216Metric
- C19, C20, C21, C27: footprint Capacitor_SMD:C_0805_2012Metric -> Capacitor_SMD:C_0402_1005Metric
- C24: value 100n -> 2u2; footprint Capacitor_SMD:C_0805_2012Metric -> Capacitor_SMD:C_1206_3216Metric
- C30: value 100n -> 1u; footprint Resistor_SMD:R_0603_1608Metric -> Capacitor_SMD:C_0805_2012Metric
- D1, D18, D19, D20, D21: value 1N5819WS -> 1N4148WS
- D10, D11, D12, D13, D14, D15, D16, D17, D2, D3, D4, D5, D6, D7, D8, D9: value 1N5819WS -> BZT52C5V6; footprint Diode_SMD:D_SOD-323 -> Diode_SMD:D_SOD-123
- Q1, Q2: value AO3400A -> SP010N01BGHTO; footprint Package_TO_SOT_SMD:SOT-23 -> Package_TO_SOT_SMD:Infineon_PG-HSOF-8-1
- Q3: value MMBT5551 -> SP010N01BGHTO; footprint Package_TO_SOT_SMD:SOT-23 -> Package_TO_SOT_SMD:Infineon_PG-HSOF-8-1
- Q4: value MMBT5401 -> SP010N01BGHTO; footprint Package_TO_SOT_SMD:SOT-23 -> Package_TO_SOT_SMD:Infineon_PG-HSOF-8-1
- Q7: value AO3400A -> CXT5551; footprint Package_TO_SOT_SMD:SOT-23 -> Package_TO_SOT_SMD:SOT-89-3
- R20, R21, R26, R30: value 4k7 -> 2k
- R22: value 4k7 -> 100
- R23: value 22 -> 8; footprint Resistor_SMD:R_1206_3216Metric -> Resistor_SMD:R_1225_3264Metric
- R27, R31: value 22 -> 100; footprint Resistor_SMD:R_1206_3216Metric -> Resistor_SMD:R_0402_1005Metric
- U1: value BQ76952 -> BQ7695202
- moved D12 182.3 mm to (259.4, 100.0)
- moved D10 180.4 mm to (259.4, 85.5)
- moved D16 173.1 mm to (246.1, 114.5)
- moved D9 172.0 mm to (246.1, 100.0)
- moved D3 169.2 mm to (246.1, 71.1)
- moved D15 164.6 mm to (246.1, 85.5)
- moved D14 163.5 mm to (246.1, 56.6)
- moved D8 163.4 mm to (246.1, 42.2)
- moved R27 159.5 mm to (257.9, 39.5)
- moved R22 154.3 mm to (257.9, 35.5)
- moved R26 154.3 mm to (257.9, 37.5)
- moved C20 149.2 mm to (244.6, 88.2)
- moved D17 144.4 mm to (217.2, 111.6)
- moved R30 136.1 mm to (229.0, 106.9)
- moved D11 135.0 mm to (203.9, 111.6)
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Connections:
- C18 pad 1: Net-(C18-Pad1) -> /REG18
- C18 pad 2: Net-(D4-K) -> GBAT
- C19 pad 1: Net-(D6-K) -> /VC12
- C19 pad 2: Net-(C19-Pad2) -> /VC13
- C20 pad 1: Net-(C20-Pad1) -> /VC13
- C20 pad 2: Net-(D3-K) -> /VC14
- C21 pad 1: Net-(D1-K) -> /VC14
- C21 pad 2: Net-(C21-Pad2) -> /VC15
- C24 pad 1: Net-(C24-Pad1) -> Net-(Q7-C)
- C24 pad 2: Net-(D13-K) -> GBAT
- C27 pad 1: Net-(C27-Pad1) -> GND
- C27 pad 2: Net-(D19-K) -> /SPL
- C30 pad 1: /CBM -> /HB
- C30 pad 2: /CBP -> /SW
- D1 pad 2: Net-(BT4--) -> VBAT
- D10 pad 2: Net-(BT3--) -> /CL8
- D11 pad 1: /CBP -> Net-(D11-K)
- D11 pad 2: Net-(D11-A) -> /CL9
- D12 pad 2: /CBM -> /CL10
- D13 pad 2: Net-(BT2--) -> /CL11
- D14 pad 1: Net-(BT1--) -> Net-(D14-K)
- D14 pad 2: Net-(D14-A) -> /CL12
- D15 pad 1: Net-(D14-A) -> Net-(D15-K)
- D15 pad 2: Net-(BT2--) -> /CL13
- D16 pad 2: Net-(BT2--) -> /CL14
- D17 pad 1: /CBP -> Net-(D17-K)
- D17 pad 2: Net-(D17-A) -> /CL15
- D18 pad 1: Net-(D18-K) -> +3V3
- D18 pad 2: /CBM -> Net-(D18-A)
- D19 pad 1: Net-(D19-K) -> /BST
- D19 pad 2: Net-(BT1--) -> +15V
- D2 pad 2: /CBM -> GBAT
- D20 pad 1: Net-(BT1-+) -> /HB
- D20 pad 2: Net-(D20-A) -> /VCCR
- D21 pad 1: Net-(D20-A) -> Net-(D21-K)
- D21 pad 2: Net-(BT1--) -> VBAT
- D3 pad 2: Net-(BT3--) -> /CL1
- D4 pad 2: Net-(BT4--) -> /CL2
- D5 pad 1: /CBP -> Net-(D5-K)
- D5 pad 2: Net-(D5-A) -> /CL3
- D6 pad 2: Net-(BT4--) -> /CL4
- D7 pad 1: Net-(BT3--) -> Net-(D7-K)
- D7 pad 2: Net-(D1-K) -> /CL5
- D8 pad 1: Net-(BT2--) -> Net-(D8-K)
- D8 pad 2: Net-(D8-A) -> /CL6
- D9 pad 1: Net-(D8-A) -> Net-(D9-K)
- D9 pad 2: Net-(BT3--) -> /CL7
- Q1 pad 1: Net-(D4-K) -> /DSG
- Q1 pad 2: Net-(BT4--) -> VBUS
- Q1 pad 3: Net-(Q1-D) -> VBAT
- Q2 pad 1: Net-(D3-K) -> /GH
- Q2 pad 2: Net-(BT3--) -> /PH
- Q3 pad 1: Net-(D6-K) -> /GD
- Q3 pad 2: Net-(BT4--) -> VBUS
- Q3 pad 3: Net-(D2-K) -> Net-(Q3-D)
- Q4 pad 1: Net-(D1-K) -> /GD
- Q4 pad 2: Net-(BT3--) -> VBUS
- Q4 pad 3: Net-(D5-A) -> Net-(Q3-D)
- Q7 pad 1: Net-(D13-K) -> /BREG
- Q7 pad 2: Net-(BT2--) -> Net-(Q7-C)
- Q7 pad 3: Net-(Q7-D) -> /REGIN
- R20 pad 1: Net-(C18-Pad1) -> /SCL
- R20 pad 2: /BAL1 -> +3V3
- R21 pad 1: Net-(C21-Pad2) -> /SDA
- R21 pad 2: /CBPE1 -> +3V3
- R22 pad 1: Net-(C20-Pad1) -> /VC4
- R22 pad 2: /BAL2 -> /CL4
- R23 pad 1: Net-(BT2--) -> /CL1
- R23 pad 2: Net-(Q2-D) -> Net-(Q16-D)
- R26 pad 1: Net-(C24-Pad1) -> /VC3
- R26 pad 2: /BAL3 -> Net-(D5-K)
- R27 pad 1: Net-(BT1--) -> /VC3
- R27 pad 2: Net-(Q7-D) -> /CL3
- R30 pad 1: Net-(C27-Pad1) -> /VC4
- R30 pad 2: /BAL4 -> Net-(D6-K)
- R31 pad 1: Net-(BT1-+) -> /VC4
- R31 pad 2: Net-(Q10-D) -> /CL4
- U1 pad 17: GND -> GBAT
- U1 pad 18: unconnected-(U1-SRP-Pad18) -> /SRP
- U1 pad 20: unconnected-(U1-SRN-Pad20) -> /SRN
- U1 pad 21: unconnected-(U1-TS1-Pad21) -> /TS1
- U1 pad 22: unconnected-(U1-TS2-Pad22) -> /WAKE
- U1 pad 23: unconnected-(U1-TS3-Pad23) -> /TS2
- U1 pad 24: unconnected-(U1-REG18-Pad24) -> /REG18
- U1 pad 25: unconnected-(U1-ALERT-Pad25) -> /ALERT
- U1 pad 26: unconnected-(U1-SCL-Pad26) -> /SCL
- U1 pad 27: unconnected-(U1-SDA-Pad27) -> /SDA
- U1 pad 28: unconnected-(U1-HDQ-Pad28) -> /TS3
- U1 pad 29: unconnected-(U1-CFETOFF-Pad29) -> /TS4
- U1 pad 30: unconnected-(U1-DFETOFF-Pad30) -> /TS5
- U1 pad 31: unconnected-(U1-DCHG-Pad31) -> /TS6
- U1 pad 32: unconnected-(U1-DDSG-Pad32) -> /TS7
- U1 pad 33: unconnected-(U1-RST_SHUT-Pad33) -> /SHUT
- U1 pad 34: unconnected-(U1-REG2-Pad34) -> GBAT
- U1 pad 35: unconnected-(U1-REG1-Pad35) -> +3V3
- U1 pad 36: unconnected-(U1-REGIN-Pad36) -> /REGIN
- U1 pad 37: unconnected-(U1-BREG-Pad37) -> /BREG
- U1 pad 38: unconnected-(U1-FUSE-Pad38) -> GBAT
- U1 pad 39: unconnected-(U1-PDSG-Pad39) -> /PDSG
- U1 pad 41: unconnected-(U1-LD-Pad41) -> /LD
- U1 pad 42: unconnected-(U1-PACK-Pad42) -> /PACK
- U1 pad 43: unconnected-(U1-DSG-Pad43) -> /DSG
- U1 pad 46: unconnected-(U1-CP1-Pad46) -> /CP
- U1 pad 47: unconnected-(U1-BAT-Pad47) -> Net-(U1-BAT)
Other:
- board outline added: 100 x 70 mm
