File: pcb/battery-pack.kicad_sch (KiCad schematic)
At the start: 47 parts, among them Q1 AO3400A, Q4 AO3401A, Q5 AO3400A, Q6 AO3400A, Q7 AO3401A, U1 BQ76952

Commit message: Save bms descrete prototype
Parts:
- removed C20: 100n, symbol Device:C
- removed D1, D2, D3: D_Schottky, symbol Device:D_Schottky
- removed Q1, Q5, Q6: AO3400A, Package_TO_SOT_SMD:SOT-23, symbol Transistor_FET:AO3400A
- removed Q4, Q7: AO3401A, Package_TO_SOT_SMD:SOT-23, symbol Transistor_FET:AO3401A
- added BT1, BT10, BT11, BT12, BT13, BT14, BT15, BT16, BT2, BT3, BT4, BT5, BT6, BT7, BT8, BT9: P45B, symbol Device:Battery_Cell
- added C19, C23, C27, C35, C36, C37, C38, C39, C40, C41, C54, C55, C56, C57, C58, C84, C85: 100n, symbol Device:C
- added C30: 100n, Resistor_SMD:R_0603_1608Metric, symbol Device:C
- added C32, C34: 10u, Resistor_SMD:R_0603_1608Metric, symbol Device:C
- added C33, C86: 1u, symbol Device:C
- added C83: C, symbol Device:C
- added D27, D30, D31, D32: 1N5819WS, Diode_SMD:D_SOD-323, symbol Diode:1N5819WS
- added L1: L, symbol Device:L
- added Q14: AO3400A, Package_TO_SOT_SMD:SOT-23, symbol Transistor_FET:AO3400A
- added Q15: MMBT5551, Package_TO_SOT_SMD:SOT-23, symbol Transistor_BJT:Q_NPN_BEC
- added Q16: NMOS, symbol Simulation_SPICE:NMOS
- added Q49: PMOS, symbol Simulation_SPICE:PMOS
- added R114, R115, R37, R38: R, Resistor_SMD:R_0402_1005Metric, symbol Device:R
- added R116: 470, symbol Device:R
- added R117: 4k7, symbol Device:R
- added R118, R34: R, symbol Device:R
- added R19, R21, R26, R27, R32, R33, R42, R43, R44, R45, R46, R47, R48, R49, R50, R51, R52, R53, R70, R71, R72, R73, R74, R75, R76, R77, R78, R79, R80, R81: 47, symbol Device:R
- added U2: LM393, Package_SO:SOIC-8_3.9x4.9mm_P1.27mm, symbol Comparator:LM393
- added U3: HT7533-1-SOT89, Package_TO_SOT_SMD:SOT-89-3, symbol Regulator_Linear:HT75xx-1-SOT89
- R18: value R -> 47
- R20: value 4k7 -> 47
Connections:
- net GND: now also C32.2, C33.2, C34.2, C83.2, C84.2, D27.2 (A), Q15.2 (E), Q16.3 (S), R38.2, U2.4 (V-), U2.5 (+), U2.6 (-), U3.1 (GND)
- net Measure1/CELLP: now reaches C18.1
- net Measure1/CELLP: now also R20.2
- net Measure1/CELLM: now reaches R18.2
- net Measure1/CELLM: now also C18.2
- net CELL1: now reaches R20.1
- net CELL1: now also BT1.2 (-), BT5.1 (+), R21.1; no longer C18.2
- net CELL0: now reaches R18.1
- net CELL0: now also BT5.2 (-)
- new net: C33.1, D31.1 (K), D32.2 (A)
- new net: C86.1, D30.1 (K), D31.2 (A)
- new net: C85.1, D32.1 (K), R117.2
- new net: C85.2, D27.1 (K), L1.1, Q14.2 (S)
- new net: R114.2, R118.2, R34.1, U2.1
- new net: R114.1, R115.2, U2.2 (-)
- new net: R37.2, R38.1, U2.3 (+)
- new net: C86.2, Q16.1 (D), Q49.1 (D)
- new net: Q14.1 (G), R116.1, R117.1
- new net: Q15.1 (B), R34.2
- new net: Q15.3 (C), R116.2
- new net +3V3: C34.1, R115.1, R118.1, U3.3 (VOUT)
- new net +5V: C32.1, C84.1, D30.2 (A), L1.2, Q49.3 (S), R37.1, U2.8 (V+), U3.2 (VIN)
- new net CBM: C30.1
- new net CBP: C30.2
- new net CELL10: BT14.2 (-), BT15.1 (+), R77.1, R78.1
- new net CELL11: BT13.2 (-), BT14.1 (+), R75.1, R76.1
- new net CELL12: BT12.2 (-), BT13.1 (+), R73.1, R74.1
- new net CELL13: BT11.2 (-), BT12.1 (+), R71.1, R72.1
- new net CELL14: BT10.2 (-), BT11.1 (+), R47.1, R70.1
- new net CELL15: BT10.1 (+), BT9.2 (-), R45.1, R46.1
- new net CELL16: BT9.1 (+), R44.1
- new net CELL2: BT1.1 (+), BT2.2 (-), R19.1, R27.1
- new net CELL3: BT2.1 (+), BT3.2 (-), R26.1, R33.1
- new net CELL4: BT3.1 (+), BT8.2 (-), R32.1, R53.1
- new net CELL5: BT7.2 (-), BT8.1 (+), R51.1, R52.1
- new net CELL6: BT6.2 (-), BT7.1 (+), R49.1, R50.1
- new net CELL7: BT4.2 (-), BT6.1 (+), R43.1, R48.1
- new net CELL8: BT16.2 (-), BT4.1 (+), R42.1, R81.1
- new net CELL9: BT15.2 (-), BT16.1 (+), R79.1, R80.1
- new net Measure10/CELLM: C57.2, R79.2
- new net Measure10/CELLP: C57.1, R78.2
- new net Measure11/CELLM: C56.2, R77.2
- new net Measure11/CELLP: C56.1, R76.2
- new net Measure12/CELLM: C55.2, R75.2
- new net Measure12/CELLP: C55.1, R74.2
- new net Measure13/CELLM: C54.2, R73.2
- new net Measure13/CELLP: C54.1, R72.2
- new net Measure14/CELLM: C38.2, R71.2
- new net Measure14/CELLP: C38.1, R70.2
- new net Measure15/CELLM: C37.2, R47.2
- new net Measure15/CELLP: C37.1, R46.2
- new net Measure16/CELLM: C36.2, R45.2
- new net Measure16/CELLP: C36.1, R44.2
- new net Measure2/CELLM: C19.2, R21.2
- new net Measure2/CELLP: C19.1, R19.2
- new net Measure3/CELLM: C23.2, R27.2
- new net Measure3/CELLP: C23.1, R26.2
- new net Measure4/CELLM: C27.2, R33.2
- new net Measure4/CELLP: C27.1, R32.2
- new net Measure5/CELLM: C41.2, R53.2
- new net Measure5/CELLP: C41.1, R52.2
- new net Measure6/CELLM: C40.2, R51.2
- new net Measure6/CELLP: C40.1, R50.2
- new net Measure7/CELLM: C39.2, R49.2
- new net Measure7/CELLP: C39.1, R48.2
- new net Measure8/CELLM: C35.2, R43.2
- new net Measure8/CELLP: C35.1, R42.2
- new net Measure9/CELLM: C58.2, R81.2
- new net Measure9/CELLP: C58.1, R80.2
- new net VBAT: C83.1, Q14.3 (D)
- no-connect marks 0 -> 1
Other:
- added sheet Balance1 (balance.kicad_sch)
- added sheet Balance10 (balance.kicad_sch)
- added sheet Balance11 (balance.kicad_sch)
- added sheet Balance12 (balance.kicad_sch)
- added sheet Balance13 (balance.kicad_sch)
- added sheet Balance14 (balance.kicad_sch)
- added sheet Balance15 (balance.kicad_sch)
- added sheet Balance16 (balance.kicad_sch)
- added sheet Balance2 (balance.kicad_sch)
- added sheet Balance3 (balance.kicad_sch)
- added sheet Balance4 (balance.kicad_sch)
- added sheet Balance5 (balance.kicad_sch)
- added sheet Balance6 (balance.kicad_sch)
- added sheet Balance7 (balance.kicad_sch)
- added sheet Balance8 (balance.kicad_sch)
- added sheet Balance9 (balance.kicad_sch)
- added sheet Measure1 (measure.kicad_sch)
- added sheet Measure10 (measure.kicad_sch)
- added sheet Measure11 (measure.kicad_sch)
- added sheet Measure12 (measure.kicad_sch)
- added sheet Measure13 (measure.kicad_sch)
- added sheet Measure14 (measure.kicad_sch)
- added sheet Measure15 (measure.kicad_sch)
- added sheet Measure16 (measure.kicad_sch)
- added sheet Measure2 (measure.kicad_sch)
- added sheet Measure3 (measure.kicad_sch)
- added sheet Measure4 (measure.kicad_sch)
- added sheet Measure5 (measure.kicad_sch)
- added sheet Measure6 (measure.kicad_sch)
- added sheet Measure7 (measure.kicad_sch)
- added sheet Measure8 (measure.kicad_sch)
- added sheet Measure9 (measure.kicad_sch)
- note added: "5ms before 90%"
- moved on the sheet: C1, C10, C11, C12, C13, C14, C15, C16, C17, C2, C3, C4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

Commit message: Save pcb
Other:
- note added: "LKS513 triple gate driver for inverter"
Changed lines of the file:
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@@
+		)
+	)
+	(text "LKS513\ntriple gate driver for inverter"
+		(exclude_from_sim no)
+		(at 40.386 89.154 0)
+		(effects
+			(font
+				(size 1.27 1.27)
+			)
 		)
 	)

Commit message: Save
Parts:
- removed D27, D30, D31, D32: 1N5819WS, Diode_SMD:D_SOD-323, symbol Diode:1N5819WS
- removed Q14: AO3400A, Package_TO_SOT_SMD:SOT-23, symbol Transistor_FET:AO3400A
- removed Q15: MMBT5551, Package_TO_SOT_SMD:SOT-23, symbol Transistor_BJT:Q_NPN_BEC
- removed Q16: NMOS, symbol Simulation_SPICE:NMOS
- removed Q49: PMOS, symbol Simulation_SPICE:PMOS
- removed R117: 4k7, symbol Device:R
- removed R118: R, symbol Device:R
- removed U2: LM393, Package_SO:SOIC-8_3.9x4.9mm_P1.27mm, symbol Comparator:LM393
- removed U3: HT7533-1-SOT89, Package_TO_SOT_SMD:SOT-89-3, symbol Regulator_Linear:HT75xx-1-SOT89
- added Q14, Q15: Q_NMOS, symbol Device:Q_NMOS
- added Q16: Q_PNP, symbol Device:Q_PNP
- added U2: LM5148, Package_DFN_QFN:Texas_RGY_R-PVQFN-N24_EP2.05x3.1mm, symbol User_Symbols:LM5148
- C32: value 10u -> 220n; footprint Resistor_SMD:R_0603_1608Metric -> (none); LCSC C19702 -> (none)
- C33, C86: value 1u -> C
- C34: value 10u -> C; footprint Resistor_SMD:R_0603_1608Metric -> (none); LCSC C19702 -> (none)
- C84, C85: value 100n -> C
- R114, R115, R37, R38: footprint Resistor_SMD:R_0402_1005Metric -> (none)
- R116: value 470 -> R
Connections:
- net +5V: now also U2.16 (VCCX); no longer C32.1, C84.1, L1.2, R37.1
- net GND: now also C85.2, C86.2, R34.2, R37.2, Q15.S, U2.1 (NC), U2.10 (PGND), U2.2 (NC), U2.22 (NC), U2.23 (NC), U2.24 (NC), U2.7 (AGND); no longer C32.2, R38.2
- net VBAT: now also Q14.D, Q16.E, U2.12 (VIN); no longer C83.1
- net at C33.1: now also C34.1, C83.1, R38.2, U2.21 (VOUT)
- net at C86.1: now also R114.1
- net at C85.1: now also R114.2, U2.5 (COMP)
- net at L1.1: now also C32.2, Q14.S, Q15.D, U2.14 (SW); no longer C85.2
- net at R34.1: now also U2.3 (CNFG); no longer R114.2
- net at R115.2: now also U2.6 (FB); no longer R114.1
- net at R38.1: now also L1.2, U2.20 (ISNS); no longer R37.2
- net at R116.2: now also Q16.B
- net +3V3: no longer names the net of R115.1
- net +3V3: now also U2.8 (VDDA); no longer C34.1
- new net: Q14.G, U2.13 (HO)
- new net: Q16.C, U2.19 (EN)
- new net: Q15.G, U2.11 (LO)
- new net: C32.1, U2.15 (CBOOT)
- new net: C84.1, U2.9 (VCC)
- new net: R37.1, U2.4 (RT)
- no-connect marks 1 -> 0
Other:
- note added: "C19100373"
- note added: "C20605920"
- note added: "C2686653"
- note added: "C2986239"
- note added: "C2987720"
- note added: "C507088"
- note added: "C5297508"
- note added: "C5464768"
- note added: "C6989639"
- note added: "sweet spot around 20mohm 20nC"

Commit message: Save
Parts:
- added U3: STM32G4A1CETx, Package_QFP:LQFP-48_7x7mm_P0.5mm, symbol MCU_ST_STM32G4:STM32G4A1CETx
Connections:
- new net: U3.23 (VSS), U3.35 (VSS), U3.47 (VSS)
Changed lines of the file:
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@@
 		(exclude_from_sim no)
 		(in_bom yes)
-		(on_board yes)
+		(on_board no)
 		(dnp no)
 		(property "Reference" "BT4"
@@
 		(exclude_from_sim no)
 		(in_bom yes)
-		(on_board yes)
+		(on_board no)
 		(dnp no)
 		(property "Reference" "BT3"
@@
 		(exclude_from_sim no)
 		(in_bom yes)
-		(on_board yes)
+		(on_board no)
 		(dnp no)
 		(property "Reference" "BT12"
@@
 		(exclude_from_sim no)
 		(in_bom yes)
-		(on_board yes)
+		(on_board no)
 		(dnp no)
 		(property "Reference" "BT10"
@@
 		(exclude_from_sim no)
 		(in_bom yes)
-		(on_board yes)
+		(on_board no)
 		(dnp no)
 		(property "Reference" "BT5"
@@
 		(exclude_from_sim no)
 		(in_bom yes)
-		(on_board yes)
+		(on_board no)
 		(dnp no)
 		(property "Reference" "BT16"
@@
 	)
 	(symbol
+		(lib_id "MCU_ST_STM32G4:STM32G4A1CETx")
+		(at 311.15 148.59 0)
+		(unit 1)
+		(exclude_from_sim no)
+		(in_bom yes)
+		(on_board yes)
+		(dnp no)
+		(fields_autoplaced yes)
+		(property "Reference" "U3"
+			(at 315.8333 189.23 0)
+			(effects
+				(font
+					(size 1.27 1.27)
+				)
+				(justify left)
+			)
+		)
+		(property "Value" "STM32G4A1CETx"
+			(at 315.8333 191.77 0)
+			(effects
+				(font
+					(size 1.27 1.27)
+				)
+				(justify left)
+			)
+		)
+		(property "Footprint" "Package_QFP:LQFP-48_7x7mm_P0.5mm"
+			(at 295.91 186.69 0)
+			(effects
+				(font
+					(size 1.27 1.27)
+				)
+				(justify right)
+				(hide yes)
+			)
+		)
+		(property "Datasheet" "https://www.st.com/resource/en/datasheet/stm32g4a1ce.pdf"
+			(at 311.15 148.59 0)
+			(effects
+				(font
+					(size 1.27 1.27)
+				)
+				(hide yes)
+			)
+		)
+		(property "Description" "STMicroelectronics Arm Cortex-M4 MCU, 512KB flash, 112KB RAM, 170 MHz, 1.71-3.6V, 38 GPIO, LQFP48"
+			(at 311.15 148.59 0)
+			(effects
+				(font
+					(size 1.27 1.27)
+				)
+				(hide yes)
+			)
+		)
+		(pin "19"
+		)
+		(pin "47"
+		)
+		(pin "37"
+		)
+		(pin "30"
+		)
+		(pin "33"
+		)
+		(pin "28"
+		)
+		(pin "1"
+		)
+		(pin "36"
+		)
+		(pin "48"
+		)
+		(pin "24"
+		)
+		(pin "29"
+		)
+		(pin "31"
+		)
+		(pin "9"
+		)
+		(pin "32"
+		)
+		(pin "23"
+		)
+		(pin "4"
+		)
+		(pin "8"
+		)
+		(pin "18"
+		)
+		(pin "25"
+		)
+		(pin "14"
+		)
+		(pin "16"
+		)
+		(pin "3"
+		)
+		(pin "2"
+		)
+		(pin "35"
+		)
+		(pin "7"
+		)
+		(pin "20"
+		)
+		(pin "45"
+		)
+		(pin "6"
+		)
+		(pin "5"
+		)
+		(pin "43"
+		)
+		(pin "40"
+		)
+		(pin "11"
+		)
+		(pin "22"
+		)
+		(pin "12"
+		)
+		(pin "26"
+		)
+		(pin "46"
+		)
+		(pin "38"
+		)
+		(pin "27"
+		)
+		(pin "15"
+		)
+		(pin "10"
+		)
+		(pin "13"
+		)
+		(pin "44"
+		)
+		(pin "21"
+		)
+		(pin "17"
+		)
+		(pin "34"
+		)
+		(pin "41"
+		)
+		(pin "39"
+		)
+		(pin "42"
+		)
+		(instances
+			(project ""
+				(path "/38b0a34b-2047-47f6-90d7-ccdf77e8e212"
+					(reference "U3")
+					(unit 1)
+				)
+			)
+		)
+	)
+	(symbol
 		(lib_id "Device:R")
 		(at 181.61 213.36 90)
@@
 		(exclude_from_sim no)
 		(in_bom yes)
-		(on_board yes)
+		(on_board no)
 		(dnp no)
 		(property "Reference" "BT8"
@@
 		(exclude_from_sim no)
 		(in_bom yes)
-		(on_board yes)
+		(on_board no)
 		(dnp no)
 		(property "Reference" "BT1"
@@
 		(exclude_from_sim no)
 		(in_bom yes)
-		(on_board yes)
+		(on_board no)
 		(dnp no)
 		(property "Reference" "BT13"
@@
 		(exclude_from_sim no)
 		(in_bom yes)
-		(on_board yes)
+		(on_board no)
 		(dnp no)
 		(property "Reference" "BT14"
@@
 		(exclude_from_sim no)
 		(in_bom yes)
-		(on_board yes)
+		(on_board no)
 		(dnp no)
 		(property "Reference" "BT11"
@@
 		(exclude_from_sim no)
 		(in_bom yes)
-		(on_board yes)
+		(on_board no)
 		(dnp no)
 		(property "Reference" "BT2"
@@
 		(exclude_from_sim no)
 		(in_bom yes)
-		(on_board yes)
+		(on_board no)
 		(dnp no)
 		(property "Reference" "BT6"
@@
 		(exclude_from_sim no)
 		(in_bom yes)
-		(on_board yes)
+		(on_board no)
 		(dnp no)
 		(property "Reference" "BT9"
@@
 		(exclude_from_sim no)
 		(in_bom yes)
-		(on_board yes)
+		(on_board no)
 		(dnp no)
 		(property "Reference" "BT15"
@@
 		(exclude_from_sim no)
 		(in_bom yes)
-		(on_board yes)
+		(on_board no)
 		(dnp no)
 		(property "Reference" "BT7"

Commit message: Save
Other:
- note removed: "2nF capacitance"
- note removed: "2x loss so 40x for 5% diff"
- note removed: "5V -> 2V in 100uS"
- note removed: "5V gate drive"
- note removed: "5ms before 90%"
- note removed: "one time constant"
- moved on the sheet: C30
Changed lines of the file:
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@@
 		)
 	)
-	(text "5V gate drive"
-		(exclude_from_sim no)
-		(at 407.924 276.86 0)
-		(effects
-			(font
-				(size 1.27 1.27)
-			)
-		)
-	)
 	(text "C507088"
 		(exclude_from_sim no)
@@
 		)
 	)
-	(text "5ms before 90%"
-		(exclude_from_sim no)
-		(at 408.94 267.716 0)
-		(effects
-			(font
-				(size 1.27 1.27)
-			)
-		)
-	)
 	(text "C2686653"
 		(exclude_from_sim no)
@@
 		)
 	)
-	(text "2x loss so 40x for 5% diff"
-		(exclude_from_sim no)
-		(at 408.432 287.274 0)
-		(effects
-			(font
-				(size 1.27 1.27)
-			)
-		)
-	)
-	(text "one time constant"
-		(exclude_from_sim no)
-		(at 408.432 273.304 0)
-		(effects
-			(font
-				(size 1.27 1.27)
-			)
-		)
-	)
 	(text "C2986239"
 		(exclude_from_sim no)
@@
 		)
 	)
-	(text "2nF capacitance"
-		(exclude_from_sim no)
-		(at 407.416 283.21 0)
-		(effects
-			(font
-				(size 1.27 1.27)
-			)
-		)
-	)
 	(text "C20605920"
 		(exclude_from_sim no)
@@
 		)
 	)
-	(text "5V -> 2V in 100uS"
-		(exclude_from_sim no)
-		(at 407.924 279.908 0)
-		(effects
-			(font
-				(size 1.27 1.27)
-			)
-		)
-	)
 	(junction
 		(at 226.06 175.26)
@@
 	(wire
 		(pts
-			(xy 377.19 259.08) (xy 377.19 256.54)
+			(xy 266.7 250.19) (xy 266.7 247.65)
 		)
 		(stroke
@@
 	(wire
 		(pts
-			(xy 377.19 256.54) (xy 382.27 256.54)
+			(xy 266.7 247.65) (xy 271.78 247.65)
 		)
 		(stroke
@@
 	(wire
 		(pts
-			(xy 377.19 269.24) (xy 382.27 269.24)
+			(xy 266.7 260.35) (xy 271.78 260.35)
 		)
 		(stroke
@@
 	(wire
 		(pts
-			(xy 377.19 266.7) (xy 377.19 269.24)
+			(xy 266.7 257.81) (xy 266.7 260.35)
 		)
 		(stroke
@@
 	)
 	(label "CBM"
-		(at 378.46 269.24 0)
+		(at 267.97 260.35 0)
 		(effects
 			(font
@@
 	)
 	(label "CBP"
-		(at 378.46 256.54 0)
+		(at 267.97 247.65 0)
 		(effects
 			(font
@@
 	(symbol
 		(lib_id "Device:C")
-		(at 377.19 262.89 0)
+		(at 266.7 254 0)
 		(mirror x)
 		(unit 1)
@@
 		(dnp no)
 		(property "Reference" "C30"
-			(at 382.905 261.493 0)
+			(at 272.415 252.603 0)
 			(effects
 				(font
@@
 		)
 		(property "Value" "100n"
-			(at 382.905 264.033 0)
+			(at 272.415 255.143 0)
 			(effects
 				(font
@@
 		)
 		(property "Footprint" "Resistor_SMD:R_0603_1608Metric"
-			(at 378.1552 259.08 0)
+			(at 267.6652 250.19 0)
 			(effects
 				(font
@@
 		)
 		(property "Datasheet" "~"
-			(at 377.19 262.89 0)
+			(at 266.7 254 0)
 			(effects
 				(font
@@
 		)
 		(property "Description" "Unpolarized capacitor"
-			(at 377.19 262.89 0)
+			(at 266.7 254 0)
 			(effects
 				(font

Commit message: Save
Parts:
- removed BT1, BT10, BT11, BT12, BT13, BT14, BT15, BT16, BT2, BT3, BT4, BT5, BT6, BT7, BT8, BT9: P45B, symbol Device:Battery_Cell
- removed C10, C11, C12, C13, C14, C15, C16, C17, C32, C6, C7, C8, C9: 220n, symbol Device:C
- removed C19, C35, C36, C37, C38, C39, C40, C41, C54, C55, C56, C57, C58: 100n, symbol Device:C
- removed C30: 100n, Resistor_SMD:R_0603_1608Metric, symbol Device:C
- removed C84, C85, C86: C, symbol Device:C
- removed L1: L, symbol Device:L
- removed Q14, Q15: Q_NMOS, symbol Device:Q_NMOS
- removed Q16: Q_PNP, symbol Device:Q_PNP
- removed R114, R115, R116, R34, R37, R38: R, symbol Device:R
- removed R13, R14, R15, R16, R17, R2, R3, R4, R5, R6: 20, symbol Device:R
- removed R26, R27, R32, R33, R42, R43, R44, R45, R46, R47, R48, R49, R50, R51, R52, R53, R70, R71, R72, R73, R74, R75, R76, R77, R78: 47, symbol Device:R
- removed U2: LM5148, Package_DFN_QFN:Texas_RGY_R-PVQFN-N24_EP2.05x3.1mm, symbol User_Symbols:LM5148
- removed U3: STM32G4A1CETx, Package_QFP:LQFP-48_7x7mm_P0.5mm, symbol MCU_ST_STM32G4:STM32G4A1CETx
- added C24, C89: 2u2, Capacitor_SMD:C_1206_3216Metric, symbol Device:C
- added C25, C52: 100n, Capacitor_SMD:C_0402_1005Metric, symbol Device:C
- added C88, C96, C97, C98: 10u, Capacitor_SMD:C_1206_3216Metric, symbol Device:C
- added C90: 100p, Capacitor_SMD:C_0402_1005Metric, symbol Device:C
- added D1, D19, D20, D21, D24, D25: 1N4148WS, Diode_SMD:D_SOD-323, symbol Diode:1N4148WS
- added D22, D23: BZT52Bxx, Diode_SMD:D_SOD-123, symbol Diode:BZT52Bxx
- added J1: Conn_01x02, symbol Connector_Generic:Conn_01x02
- added J10: Conn_01x02, User_Footprints:1x02_2.00mm_Solder, symbol Connector_Generic:Conn_01x02
- added L3: 20u, symbol Device:L
- added Q1, Q2, Q21, Q3, Q4, Q5, Q6, Q8: SP010N01BGHTO, Package_TO_SOT_SMD:Infineon_PG-HSOF-8-1, symbol User_Symbols:SP010N01BGHTO
- added Q10, Q9: Q_NMOS_GSD, symbol Transistor_FET:Q_NMOS_GSD
- added Q24: AGM150P10D, Package_TO_SOT_SMD:TO-252-2, symbol Device:Q_PMOS
- added Q7: CXT5551, Package_TO_SOT_SMD:SOT-89-3, symbol Transistor_BJT:Q_NPN_BCE
- added R100, R107, R110, R111, R112: 1M, Resistor_SMD:R_0402_1005Metric, symbol Device:R
- added R101, R98: 1m, User_Footprints:R_Shunt_3921, symbol Device:R
- added R102, R103: 1, Resistor_SMD:R_0603_1608Metric, symbol Device:R
- added R108, R109, R82, R83, R84, R90: 2k, Resistor_SMD:R_0402_1005Metric, symbol Device:R
- added R85, R86, R87, R88, R89: 100, Resistor_SMD:R_0402_1005Metric, symbol Device:R
- added R99: 0.5, symbol Device:R
- added TH1, TH2: 10k, symbol Device:Thermistor
- added U3, U8: IRS2181STR, Package_SO:JEITA_SOIC-8_3.9x4.9mm_P1.27mm, symbol User_Symbols:IRS2181STR
- added U4: STM32C011F6Px, Package_SO:TSSOP-20_4.4x6.5mm_P0.65mm, symbol MCU_ST_STM32C0:STM32C011F6Px
- added U6: SP485E, Package_SO:JEITA_SOIC-8_3.9x4.9mm_P1.27mm, symbol User_Symbols:SP485E
- C1: value 220n -> 100n; footprint (none) -> Capacitor_SMD:C_0402_1005Metric; LCSC (none) -> C1525
- C18: value 100n -> 10u; footprint (none) -> Capacitor_SMD:C_1206_3216Metric; LCSC (none) -> C380364
- C2, C4: value 220n -> 100p; footprint (none) -> Capacitor_SMD:C_0402_1005Metric; LCSC (none) -> C1546
- C23: value 100n -> 1u; footprint (none) -> Capacitor_SMD:C_0805_2012Metric; LCSC (none) -> C28323
- C27: footprint (none) -> Capacitor_SMD:C_0402_1005Metric; LCSC (none) -> C307331
- C3: value 220n -> 1u; footprint (none) -> Capacitor_SMD:C_0805_2012Metric; LCSC (none) -> C28323
- C33, C34: value C -> 10u; footprint (none) -> Capacitor_SMD:C_1206_3216Metric; LCSC (none) -> C380364
- C5: value 220n -> 2u2; footprint (none) -> Capacitor_SMD:C_1206_3216Metric; LCSC (none) -> C920964
- C83: value C -> 100u; now not fitted
- R1, R11, R12: value 20 -> 100; footprint (none) -> Resistor_SMD:R_0402_1005Metric; LCSC (none) -> C25076
- R10: value 20 -> 2k; footprint (none) -> Resistor_SMD:R_0402_1005Metric; LCSC (none) -> C4109
- R18: value 47 -> 1m
- R19, R20, R21, R81: value 47 -> 2k; footprint (none) -> Resistor_SMD:R_0402_1005Metric; LCSC (none) -> C4109
- R7, R8: value 20 -> 1m
- R79: value 47 -> 15; now not fitted
- R80: value 47 -> 1M; footprint (none) -> Resistor_SMD:R_0402_1005Metric; LCSC (none) -> C26083
- R9: value 20 -> 1M; footprint (none) -> Resistor_SMD:R_0402_1005Metric; LCSC (none) -> C26083
- U1: value BQ76952 -> BQ7695202; LCSC (none) -> C3038665
Connections:
- net CELL0 is gone; now on net GBAT: R18.1
- net CELL2 is gone; now on net PDSG: R19.1
- net CELL8 is gone; now on net PACK: R81.1
- net Measure2/CELLM is gone; now on net +3V3: R21.2
- net Measure2/CELLP is gone; now on an unnamed net: R19.2
- net Measure3/CELLM is gone; now on net GBAT: C23.2
- net Measure3/CELLP is gone; now on net +3V3: C23.1
- net Measure4/CELLP is gone; now on net GND: C27.1
- net Measure9/CELLP is gone; now on net GBAT: R80.2
- net +5V: now also C52.2, U6.8 (VCC)
- net GND: now also R12.2, R18.2, R7.2, R8.2, C52.1, C88.2, C98.2, Q10.2 (S), Q6.2 (S), R112.2, R99.2, U3.2 (INL), U3.3 (COM), U4.5 (VSS), U6.5 (GND), U8.3 (COM); no longer C33.2, U1.17 (VSS)
- net VBAT: now also R9.2, C89.2, D1.2 (A), D21.2 (A), D23.1 (K), Q1.3 (D), Q21.3 (D), Q24.S, Q8.3 (D)
- net VC10: no longer R7.2
- net VC11: no longer C5.2
- net VC12: no longer C4.2, C5.1
- net VC13: no longer C3.2, C4.1
- net VC14: no longer C2.2, C3.1
- net VC15: no longer C1.2, C2.1
- net VC16: no longer C1.1, R1.2
- net VC5: no longer R12.2
- net VC6: no longer R11.2
- net VC7: no longer R10.2
- net VC8: no longer R9.2
- net VC9: no longer R8.2
- net SRP: now reaches R11.1
- net SRP: now also C1.2, C2.2, U1.18 (SRP)
- net PDGATE: now reaches R9.1
- net PDGATE: now also R10.2, D23.2 (A), Q24.G
- net GBAT: now reaches R8.1
- net GBAT: now also C18.2, C5.2, R11.2, R7.1, U1.17 (VSS), U1.34 (REG2), U1.38 (FUSE), C24.2, C25.1, C90.1, R90.1, TH1.2, TH2.2
- net at R1.1: now also D1.1 (K)
- net SRN: now reaches U1.20 (SRN)
- net SRN: now also C1.1, C2.1, R12.1
- net TS1: now reaches U1.21 (TS1)
- net TS1: now also TH1.1
- net WAKE: now reaches U1.22 (TS2)
- net WAKE: now also J1.1 (Pin_1)
- net TS2: now reaches U1.23 (TS3)
- net TS2: now also TH2.1
- net REG18: now reaches U1.24 (REG18)
- net REG18: now also C18.1
- net ALERT: now reaches U1.25 (ALERT)
- net SCL: now reaches U1.26 (SCL)
- net SCL: now also R20.1
- net SDA: now reaches U1.27 (SDA)
- net SDA: now also R21.1
- net TS3: now reaches U1.28 (HDQ)
- net TS4: now reaches U1.29 (CFETOFF)
- net TS5: now reaches U1.30 (DFETOFF)
- net TS6: now reaches U1.31 (DCHG)
- net TS7: now reaches U1.32 (DDSG)
- net SHUT: now reaches U1.33 (RST_SHUT)
- net +3V3: now reaches U1.35 (REG1)
- net +3V3: now also R20.2, D20.1 (K), U4.4 (VDD)
- net REGIN: now reaches U1.36 (REGIN)
- net REGIN: now also C25.2, Q7.3 (E)
- net BREG: now reaches U1.37 (BREG)
- net BREG: now also Q7.1 (B)
- net PDSG: now reaches U1.39 (PDSG)
- net LD: now reaches U1.41 (LD)
- net LD: now also R82.1
- net PACK: now reaches U1.42 (PACK)
- net DSG: now reaches U1.43 (DSG)
- net DSG: now also R109.1
- net CP: now reaches U1.46 (CP1)
- net CP: now also C3.1
- net BAT: now reaches U1.47 (BAT)
- net BAT: now also C3.2, C4.2, C5.1, R1.2, R110.1
- removed net CELL1: R20.1, R21.1
- net CELL9: no longer names the net of R80.1
- net CELL9: now also C4.1, C90.2, R110.2; no longer R79.1
- removed net Measure1/CELLM: C18.2, R18.2
- removed net Measure1/CELLP: C18.1, R20.2
- net Measure10/CELLM renamed VPRE
- net VPRE: now also Q24.D
- net Measure4/CELLM renamed SPL
- net SPL: now also R86.2, R87.2, R88.1, R89.1
- net Measure9/CELLM: no longer names the net of R81.2
- net Measure9/CELLM: now also R84.1
- new net: C97.1, D24.2 (A), D25.1 (K)
- new net: C83.1, Q2.3 (D), Q5.3 (D), R101.2, R98.2
- new net: J1.2 (Pin_2), R90.2
- new net: C24.1, Q7.2 (C), R85.2
- new net: D21.1 (K), R85.1
- new net: R82.2, R83.1
- new net: C97.2, Q10.3 (D), Q9.2 (S)
- new net: L3.1, Q3.3 (D), Q4.3 (D)
- new net: L3.2, R101.1, R98.1
- new net: R108.1, R109.2
- new net +15V: C34.1, C88.1, C98.1, D19.2 (A), D25.2 (A), U3.5 (VCC), U8.5 (VCC)
- new net BST: C33.1, D19.1 (K), U8.8 (VB)
- new net DEN: U6.3 (DE)
- new net DGATE: D22.1 (K), Q1.1 (G), Q21.1 (G), Q8.1 (G), R107.2, R108.2
- new net GCH: R103.1, U8.7 (HO)
- new net GCL: R102.1, U8.4 (LO)
- new net GD: Q3.1 (G), Q4.1 (G), R100.2, U3.7 (HO)
- new net GH: Q2.1 (G), Q5.1 (G), R103.2, R111.1
- new net GL: Q6.1 (G), R102.2, R112.1
- new net INFL: U8.2 (INL)
- new net INLD: U8.1 (INH)
- new net INREC: U3.1 (INH)
- new net Logic Power/3V3: D20.2 (A)
- new net PH: C33.2, Q2.2 (S), Q5.2 (S), Q6.3 (D), R111.2, R99.1, U8.6 (VS)
- new net REN: U6.2 (~{RE})
- new net RSA: J10.2 (Pin_2), R88.2, R89.2, U6.6 (A)
- new net RSB: J10.1 (Pin_1), R86.1, R87.1, U6.7 (B)
- new net RX: U6.1 (RO)
- new net TX: U6.4 (DI)
- new net VBST: C96.1, D24.1 (K), U3.8 (VB)
- new net VBUS: C89.1, C96.2, D22.2 (A), Q1.2 (S), Q21.2 (S), Q3.2 (S), Q4.2 (S), Q8.2 (S), Q9.3 (D), R100.1, R107.1, R79.1, R83.2, R84.2, U3.6 (VS)
- no-connect marks 0 -> 3
Other:
- removed sheet Balance1
- removed sheet Balance10
- removed sheet Balance11
- removed sheet Balance12
- removed sheet Balance13
- removed sheet Balance14
- removed sheet Balance15
- removed sheet Balance16
- removed sheet Balance2
- removed sheet Balance3
- removed sheet Balance4
- removed sheet Balance5
- removed sheet Balance6
- removed sheet Balance7
- removed sheet Balance8
- removed sheet Balance9
- removed sheet Measure1
- removed sheet Measure10
- removed sheet Measure11
- removed sheet Measure12
- removed sheet Measure13
- removed sheet Measure14
- removed sheet Measure15
- removed sheet Measure16
- removed sheet Measure2
- removed sheet Measure3
- removed sheet Measure4
- removed sheet Measure5
- removed sheet Measure6
- removed sheet Measure7
- removed sheet Measure8
- removed sheet Measure9
- added sheet Aux (aux-power.kicad_sch)
- added sheet Cell0 (cell.kicad_sch)
- added sheet Cell1 (cell.kicad_sch)
- added sheet Cell10 (cell.kicad_sch)
- added sheet Cell11 (cell.kicad_sch)
- added sheet Cell12 (cell.kicad_sch)
- added sheet Cell13 (cell.kicad_sch)
- added sheet Cell14 (cell.kicad_sch)
- added sheet Cell15 (cell.kicad_sch)
- added sheet Cell2 (cell.kicad_sch)
- added sheet Cell3 (cell.kicad_sch)
- added sheet Cell4 (cell.kicad_sch)
- added sheet Cell5 (cell.kicad_sch)
- added sheet Cell6 (cell.kicad_sch)
- added sheet Cell7 (cell.kicad_sch)
- added sheet Cell8 (cell.kicad_sch)
- added sheet Cell9 (cell.kicad_sch)
- added sheet Logic Power (logic-power.kicad_sch)
- added sheet Regen (regen.kicad_sch)
- note added: "25mA max"
- note added: "3us/A"
- note added: "FIX DIODES"
- note added: "Some negative current protection?"
- note added: "close if capacitor voltage too high"
- note removed: "C19100373"
- note removed: "C20605920"
- note removed: "C2686653"
- note removed: "C2986239"
- note removed: "C2987720"
- note removed: "C507088"
- note removed: "C5297508"
- note removed: "C5464768"
- note removed: "C6989639"
- note removed: "LKS513 triple gate driver for inverter"
- note removed: "sweet spot around 20mohm 20nC"
- moved on the sheet: U1
